File: PCB/RCSMCtrl.sch (KiCad schematic (older format))
At the start: 36 parts, among them IC1 PIC12(L)F1822-I/P, K1 RELAY_2RT, K2 RELAY_2RT, P1 CONN_01X15, P2 CONN_01X03, Q1 Q_NPN_EBC, Q2 Q_PNP_EBC, Q3 Q_NPN_EBC, SW1 SW_PUSH, SW2 SW_PUSH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

Commit message: Here it is
Parts:
- C2: value CP1_Small -> 33uF
- D7, D8: value D -> SMA
- IC1: value PIC12(L)F1822-I/P -> PIC12F1822-I/P
- Q1, Q3: value Q_NPN_EBC -> 2N7000
- Q2: value Q_PNP_EBC -> 2N3906
- R1, R12, R5, R6, R7, R9: value R -> 47K
- R10, R13, R2, R3, R8: value R -> 1K
- R11: value R -> 220R
- R4: value R -> 10K
Changed lines of the file:
@@
 P 3900 4900
 F 0 "IC1" H 2650 5450 50  0000 L CNN
-F 1 "PIC12(L)F1822-I/P" H 2650 5350 50  0000 L CNN
+F 1 "PIC12F1822-I/P" H 2650 5350 50  0000 L CNN
 F 2 "Housings_DIP:DIP-8_W7.62mm" H 3900 4900 60  0001 C CNN
 F 3 "" H 3900 4900 60  0000 C CNN
@@
 P 7700 1400
 F 0 "C2" H 7710 1470 50  0000 L CNN
-F 1 "CP1_Small" H 7710 1320 50  0000 L CNN
+F 1 "33uF" H 7710 1320 50  0000 L CNN
 F 2 "Capacitors_Elko_ThroughHole:Elko_vert_11.2x6.3mm_RM2.5_CopperClear" H 7700 1400 60  0001 C CNN
 F 3 "" H 7700 1400 60  0000 C CNN
@@
 F 0 "U1" H 8000 1450 40  0000 C CNN
 F 1 "LM7805CT" H 8200 1450 40  0000 L CNN
-F 2 "Power_Integrations:TO-220" H 8200 1350 30  0000 C CIN
+F 2 "Power_Integrations:TO-220" H 8200 1350 30  0001 C CIN
 F 3 "" H 8200 1250 60  0000 C CNN
 	1    8200 1250
@@
 P 6950 4800
 F 0 "R11" V 7030 4800 50  0000 C CNN
-F 1 "R" V 6950 4800 50  0000 C CNN
+F 1 "220R" V 6950 4800 50  0000 C CNN
 F 2 "Resistors_SMD:R_0805_HandSoldering" V 6880 4800 30  0001 C CNN
 F 3 "" H 6950 4800 30  0000 C CNN
@@
 P 4850 2400
 F 0 "R2" V 4930 2400 50  0000 C CNN
-F 1 "R" V 4850 2400 50  0000 C CNN
+F 1 "1K" V 4850 2400 50  0000 C CNN
 F 2 "Resistors_SMD:R_0805_HandSoldering" V 4780 2400 30  0001 C CNN
 F 3 "" H 4850 2400 30  0000 C CNN
@@
 P 5300 2400
 F 0 "R4" V 5380 2400 50  0000 C CNN
-F 1 "R" V 5300 2400 50  0000 C CNN
+F 1 "10K" V 5300 2400 50  0000 C CNN
 F 2 "Resistors_SMD:R_0805_HandSoldering" V 5230 2400 30  0001 C CNN
 F 3 "" H 5300 2400 30  0000 C CNN
@@
 P 5650 2100
 F 0 "R5" V 5730 2100 50  0000 C CNN
-F 1 "R" V 5650 2100 50  0000 C CNN
+F 1 "47K" V 5650 2100 50  0000 C CNN
 F 2 "Resistors_SMD:R_0805_HandSoldering" V 5580 2100 30  0001 C CNN
 F 3 "" H 5650 2100 30  0000 C CNN
@@
 P 4550 3900
 F 0 "Q1" H 4850 3950 50  0000 R CNN
-F 1 "Q_NPN_EBC" H 5150 3850 50  0000 R CNN
+F 1 "2N7000" H 5050 3850 50  0000 R CNN
 F 2 "Housings_TO-92:TO-92_Inline_Narrow_Oval" H 4750 4000 29  0001 C CNN
 F 3 "" H 4550 3900 60  0000 C CNN
@@
 P 5800 2400
 F 0 "Q2" H 6100 2450 50  0000 R CNN
-F 1 "Q_PNP_EBC" H 6400 2350 50  0000 R CNN
+F 1 "2N3906" H 6300 2350 50  0000 R CNN
 F 2 "Housings_TO-92:TO-92_Inline_Narrow_Oval" H 6000 2500 29  0001 C CNN
 F 3 "" H 5800 2400 60  0000 C CNN
@@
 P 6250 2700
 F 0 "R6" V 6330 2700 50  0000 C CNN
-F 1 "R" V 6250 2700 50  0000 C CNN
+F 1 "47K" V 6250 2700 50  0000 C CNN
 F 2 "Resistors_SMD:R_0805_HandSoldering" V 6180 2700 30  0001 C CNN
 F 3 "" H 6250 2700 30  0000 C CNN
@@
 P 6450 5500
 F 0 "R8" V 6530 5500 50  0000 C CNN
-F 1 "R" V 6450 5500 50  0000 C CNN
+F 1 "1K" V 6450 5500 50  0000 C CNN
 F 2 "Resistors_SMD:R_0805_HandSoldering" V 6380 5500 30  0001 C CNN
 F 3 "" H 6450 5500 30  0000 C CNN
@@
 P 6450 6100
 F 0 "R10" V 6530 6100 50  0000 C CNN
-F 1 "R" V 6450 6100 50  0000 C CNN
+F 1 "1K" V 6450 6100 50  0000 C CNN
 F 2 "Resistors_SMD:R_0805_HandSoldering" V 6380 6100 30  0001 C CNN
 F 3 "" H 6450 6100 30  0000 C CNN
@@
 P 6450 5350
 F 0 "R7" V 6530 5350 50  0000 C CNN
-F 1 "R" V 6450 5350 50  0000 C CNN
+F 1 "47K" V 6450 5350 50  0000 C CNN
 F 2 "Resistors_SMD:R_0805_HandSoldering" V 6380 5350 30  0001 C CNN
 F 3 "" H 6450 5350 30  0000 C CNN
@@
 P 6450 5950
 F 0 "R9" V 6530 5950 50  0000 C CNN
-F 1 "R" V 6450 5950 50  0000 C CNN
+F 1 "47K" V 6450 5950 50  0000 C CNN
 F 2 "Resistors_SMD:R_0805_HandSoldering" V 6380 5950 30  0001 C CNN
 F 3 "" H 6450 5950 30  0000 C CNN
@@
 P 5050 3900
 F 0 "R3" V 5130 3900 50  0000 C CNN
-F 1 "R" V 5050 3900 50  0000 C CNN
+F 1 "1K" V 5050 3900 50  0000 C CNN
 F 2 "Resistors_SMD:R_0805_HandSoldering" V 4980 3900 30  0001 C CNN
 F 3 "" H 5050 3900 30  0000 C CNN
@@
 P 4650 4200
 F 0 "R1" V 4730 4200 50  0000 C CNN
-F 1 "R" V 4650 4200 50  0000 C CNN
+F 1 "47K" V 4650 4200 50  0000 C CNN
 F 2 "Resistors_SMD:R_0805_HandSoldering" V 4580 4200 30  0001 C CNN
 F 3 "" H 4650 4200 30  0000 C CNN
@@
 P 8600 3150
 F 0 "Q3" H 8900 3200 50  0000 R CNN
-F 1 "Q_NPN_EBC" H 9200 3100 50  0000 R CNN
+F 1 "2N7000" H 9100 3100 50  0000 R CNN
 F 2 "Housings_TO-92:TO-92_Inline_Narrow_Oval" H 8800 3250 29  0001 C CNN
 F 3 "" H 8600 3150 60  0000 C CNN
@@
 P 7650 2700
 F 0 "D7" H 7650 2800 50  0000 C CNN
-F 1 "D" H 7650 2600 50  0000 C CNN
+F 1 "SMA" H 7650 2600 50  0000 C CNN
 F 2 "Diodes_SMD:Diode-SMA_Handsoldering" H 7650 2700 60  0001 C CNN
 F 3 "" H 7650 2700 60  0000 C CNN
@@
 P 7650 3200
 F 0 "D8" H 7650 3300 50  0000 C CNN
-F 1 "D" H 7650 3100 50  0000 C CNN
+F 1 "SMA" H 7650 3100 50  0000 C CNN
 F 2 "Diodes_SMD:Diode-SMA_Handsoldering" H 7650 3200 60  0001 C CNN
 F 3 "" H 7650 3200 60  0000 C CNN
@@
 P 9100 3150
 F 0 "R13" V 9180 3150 50  0000 C CNN
-F 1 "R" V 9100 3150 50  0000 C CNN
+F 1 "1K" V 9100 3150 50  0000 C CNN
 F 2 "Resistors_SMD:R_0805_HandSoldering" V 9030 3150 30  0001 C CNN
 F 3 "" H 9100 3150 30  0000 C CNN
@@
 P 8700 3450
 F 0 "R12" V 8780 3450 50  0000 C CNN
-F 1 "R" V 8700 3450 50  0000 C CNN
+F 1 "47K" V 8700 3450 50  0000 C CNN
 F 2 "Resistors_SMD:R_0805_HandSoldering" V 8630 3450 30  0001 C CNN
 F 3 "" H 8700 3450 30  0000 C CNN
