File: PCB G2R Rev A/RCSMCtrl.sch (KiCad schematic (older format))
At the start: 36 parts, among them IC1 PIC12F1822-I/P, K1 IM00, K2 IM00, P1 CONN_01X15, P2 CONN_01X03, Q1 2N7000, Q2 2N3906, Q3 2N7000, SW1 SW_PUSH, SW2 SW_PUSH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

Commit message: Update 7/15
Parts:
- removed K1, K2: IM00, Relays_THT:Relay_DPDT_Panasonic_JW2, symbol IM00
- removed P1: CONN_01X15, Wires:Wires_AWG20x15, symbol CONN_01X15
- removed P2: CONN_01X03, Pin_Headers:Pin_Header_Straight_1x03, symbol CONN_01X03
- removed SW1, SW2: SW_PUSH, Buttons_Switches_SMD:SW_SPST_PTS645, symbol SW_PUSH
- removed U1: LM7805CT, TO_SOT_Packages_SMD:TO-252-2, symbol LM7805CT
- added K1, K2: IM00, symbol Relay:IM00
- added P1: Conn_01x15, symbol Connector_Generic:Conn_01x15
- added P2: Conn_01x03, symbol Connector_Generic:Conn_01x03
- added SW1, SW2: SW_Push, symbol Switch:SW_Push
- added U1: L7805, symbol Regulator_Linear:L7805
- C1, C3, C4: symbol C_Small -> Device:C_Small
- C2: symbol CP1_Small -> Device:CP1_Small
- D1, D2, D3, D4, D7, D8: symbol D -> Device:D
- D5, D6: symbol LED -> Device:LED
- IC1: symbol PIC12(L)F1822-I/P -> RCSMCtrl-rescue:PIC12(L)F1822-I_P
- Q1, Q3: symbol Q_NPN_EBC -> Device:Q_NPN_EBC
- Q2: symbol Q_PNP_EBC -> Device:Q_PNP_EBC
- R1, R10, R11, R12, R13, R2, R3, R4, R5, R6, R7, R8, R9: symbol R -> Device:R
Connections:
- net +24V: now also K1.8, K2.8, U1.1 (IN)
- net +5V: now also P2.2 (Pin_2), U1.3 (OUT)
- net GND: now also P1.2 (Pin_2), P2.3 (Pin_3), SW1.2, SW2.2, U1.2 (GND)
- net at IC1.3 (CLKR/C1IN1-/T1OSO/CLKOUT/OSC2/CPS3/AN3/RA4), R10.2, R9.2: now also SW2.1
- net at IC1.5 (CPS2/C1OUT/SRQ/T0CKI/FLT0/SDA/SDI/INT/MDCIN1/AN2/RA2), R7.2, R8.2: now also SW1.1
- net at D4.2 (A): now also K2.3, P1.1 (Pin_1)
- net at D3.1 (K): now also P1.3 (Pin_3)
- net at D7.2 (A), D8.1 (K), Q3.3 (C): now also P1.4 (Pin_4)
- net at R11.1: now also P2.1 (Pin_1)
- net at D1.2 (A), D2.1 (K), Q1.3 (C): now also K1.1, K2.1
- new net: K1.2, P1.7 (Pin_7)
- new net: K1.3, P1.8 (Pin_8)
- new net: K1.4, P1.9 (Pin_9)
- new net: K1.5, P1.12 (Pin_12)
- new net: K1.6, P1.11 (Pin_11)
- new net: K1.7, P1.10 (Pin_10)
- new net: K2.4, P1.5 (Pin_5)
- new net: K2.5, P1.15 (Pin_15)
- new net: K2.6, P1.14 (Pin_14)
- new net: K2.7, P1.13 (Pin_13)
