File: PCB Mini/RCSMCtrl.kicad_pcb (KiCad board)
At the start: 2 copper layers, 58.4 x 47 mm, 37 parts, among them IC1 PIC12F1822-I/P, K1 IM00, P1 Conn_01x10, P2 CONN_01X03, Q1 2N7000, Q2 2N3906, Q3 2N7000, SW1 SW_PUSH, SW2 SW_PUSH, U1 LM7805CT

Commit message: mini rev A
Parts:
- added P3: CONN_01X03, Connector_PinHeader_2.54mm:PinHeader_1x03_P2.54mm_Vertical, F.Cu at (71.1, 45.1)
Routing:
- net Net-(IC1-Pad3): track 37.9 -> 74.4 mm, vias 1 -> 2
- net Net-(IC1-Pad5): track 60.9 -> 73.8 mm, vias 1 -> 2
- net Net-(K1-Pad3): track 19.9 -> 28.2 mm
- net GND: track 175.0 -> 181.0 mm
- net Net-(K1-Pad4): track 19.4 -> 21.9 mm
- net Net-(D7-Pad2): track 61.9 -> 63.9 mm
- added copper zone on F.Cu, net GND
Other:
- board text added: "Remote"
- board text added: "Rev. A"
- board text added: "Servo"
- board text removed: "Rev. n/c"
