File: PCB G2R Rev B/RCSMCtrl.kicad_pcb (KiCad board)
At the start: 2 copper layers, 53.3 x 58.4 mm, 41 parts, among them IC1 PIC12F1822-I/P, K1 IM00, K2 IM00, P1 Conn_01x15, P2 Conn_01x03, P3 Conn_01x03, Q1 2N7000, Q2 2N3906, Q3 2N7000, SW1 SW_Push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

Commit message: Fixed for MacroPIC
Other:
- net class Default removed
